Commit message: correction for wheel seperation

File: description/gazebo_control.xacro (robot description, xacro)
@@ -6,5 +6,5 @@
             <left_joint>left_wheel_joint</left_joint>
             <right_joint>right_wheel_joint</right_joint>
-            <wheel_separation>0.10206</wheel_separation>
+            <wheel_separation>0.10223</wheel_separation>
             <wheel_diameter>0.045</wheel_diameter>
             <!-- Limits-->

File: description/robot_core.xacro (robot description, xacro)
@@ -50,5 +50,5 @@
         <parent link="base_link"/>
         <child link="left_wheel"/>
-        <origin xyz="0 0.05103 0" rpy="-${pi/2} 0 0"/>
+        <origin xyz="0 0.05113 0" rpy="-${pi/2} 0 0"/>
         <axis xyz="0.0 0.0 1"/>
     </joint>
@@ -73,5 +73,5 @@
         <parent link="base_link"/>
         <child link="right_wheel"/>
-        <origin xyz="0 -0.05103 0" rpy="${pi/2} 0 0"/>
+        <origin xyz="0 -0.05113 0" rpy="${pi/2} 0 0"/>
         <axis xyz="0.0 0.0 -1"/>
     </joint>
