Commit message: camera_test_dev

File: description/camera.xacro (robot description, xacro)
@@ -4,5 +4,5 @@
         <parent link="chassis"/>
         <child link="camera_link"/>
-        <origin xyz="0.14688 0 59.16" rpy="0 0 0"/>
+        <origin xyz="0.14688 0 0.05916" rpy="0 0 0"/>
     </joint>
     <link name="camera_link">
@@ -31,29 +31,24 @@
     </link>
      <gazebo reference="camera_link">
-        <!-- <sensor name="laser" type="ray">
+        <sensor name="camera" type="camera">
             <pose> 0 0 0 0 0 0 </pose>
             <visualize>true</visualize>
             <update_rate>10</update_rate>
-            <ray>
-                <scan>
-                    <horizontal>
-                        <samples>360</samples>
-                        <min_angle>-3.12763</min_angle>
-                        <max_angle>3.12763</max_angle>
-                    </horizontal>
-                </scan>
-                <range>
-                    <min>0.02</min>
-                    <max>12</max>
-                </range>
-            </ray>
-            <plugin name="laser_controller" filename="libgazebo_ros_ray_sensor.so">
-                <ros>
-                    <argument>~/out:=scan</argument>
-                </ros>
-                <output_type>sensor_msgs/LaserScan</output_type>
-                <frame_name>laser_frame</frame_name>
+            <camera>
+                <horizontal_fov>1.5708</horizontal_fov>
+                <image>
+                    <format>R8G8B8</format>
+                    <width>1920</width>
+                    <height>1080</height>
+                </image>
+                <clip>
+                    <near>0.05</near>
+                    <far>8.0</far>
+                </clip>
+            </camera>
+            <plugin name="camera_controller" filename="libgazebo_ros_camera.so">
+                <frame_name>camera_link_optical</frame_name>
             </plugin>
-        </sensor> -->
+        </sensor>
     </gazebo>
 </robot>
