Commit message: ld19

File: description/ld19.xacro (robot description, xacro)
@@ -3,8 +3,8 @@
     <joint name="laser_joint" type="fixed">
         <parent link="chassis"/>
-        <child link="base_link"/>
+        <child link="laser_frame"/>
         <origin xyz="0.07725 0 0.10009" rpy="0 0 ${pi/2}"/>
     </joint>
-    <link name="base_link">
+    <link name="laser_frame">
         <visual>
             <geometry>
@@ -22,5 +22,5 @@
         </xacro:inertial_cylinder>
     </link>
-     <!-- <gazebo reference="base_link">
+     <!-- <gazebo reference="laser_frame">
         <sensor name="laser" type="ray">
             <pose> 0 0 0 0 0 0 </pose>
@@ -45,5 +45,5 @@
                 </ros>
                 <output_type>sensor_msgs/LaserScan</output_type>
-                <frame_name>base_link</frame_name>
+                <frame_name>laser_frame</frame_name>
             </plugin>
         </sensor>

Commit message: ld19 test on rasp

File: description/ld19.xacro (robot description, xacro)
@@ -3,8 +3,8 @@
     <joint name="laser_joint" type="fixed">
         <parent link="chassis"/>
-        <child link="laser_frame"/>
+        <child link="base_laser"/>
         <origin xyz="0.07725 0 0.10009" rpy="0 0 ${pi/2}"/>
     </joint>
-    <link name="laser_frame">
+    <link name="base_laser">
         <visual>
             <geometry>
@@ -22,5 +22,5 @@
         </xacro:inertial_cylinder>
     </link>
-     <!-- <gazebo reference="laser_frame">
+     <!-- <gazebo reference="base_laser">
         <sensor name="laser" type="ray">
             <pose> 0 0 0 0 0 0 </pose>
@@ -45,5 +45,5 @@
                 </ros>
                 <output_type>sensor_msgs/LaserScan</output_type>
-                <frame_name>laser_frame</frame_name>
+                <frame_name>base_laser</frame_name>
             </plugin>
         </sensor>

Commit message: test 1

File: description/ld19.xacro (robot description, xacro)
@@ -1,10 +1,10 @@
 <?xml version="1.0"?>
 <robot xmlns:xacro="http://www.ros.org/wiki/xacro"  name="robot">
-    <joint name="laser_joint" type="fixed">
+    <joint name="base_laser" type="fixed">
         <parent link="chassis"/>
-        <child link="base_laser"/>
+        <child link="laser_frame"/>
         <origin xyz="0.07725 0 0.10009" rpy="0 0 ${pi/2}"/>
     </joint>
-    <link name="base_laser">
+    <link name="laser_frame">
         <visual>
             <geometry>
@@ -22,5 +22,5 @@
         </xacro:inertial_cylinder>
     </link>
-     <!-- <gazebo reference="base_laser">
+     <!-- <gazebo reference="laser_frame">
         <sensor name="laser" type="ray">
             <pose> 0 0 0 0 0 0 </pose>
@@ -45,5 +45,5 @@
                 </ros>
                 <output_type>sensor_msgs/LaserScan</output_type>
-                <frame_name>base_laser</frame_name>
+                <frame_name>laser_frame</frame_name>
             </plugin>
         </sensor>

Commit message: test2

File: description/ld19.xacro (robot description, xacro)
@@ -1,10 +1,10 @@
 <?xml version="1.0"?>
 <robot xmlns:xacro="http://www.ros.org/wiki/xacro"  name="robot">
-    <joint name="base_laser" type="fixed">
+    <joint name="laser_joint" type="fixed">
         <parent link="chassis"/>
-        <child link="laser_frame"/>
+        <child link="base_laser"/>
         <origin xyz="0.07725 0 0.10009" rpy="0 0 ${pi/2}"/>
     </joint>
-    <link name="laser_frame">
+    <link name="base_laser">
         <visual>
             <geometry>
@@ -22,5 +22,5 @@
         </xacro:inertial_cylinder>
     </link>
-     <!-- <gazebo reference="laser_frame">
+     <!-- <gazebo reference="base_laser">
         <sensor name="laser" type="ray">
             <pose> 0 0 0 0 0 0 </pose>
@@ -45,5 +45,5 @@
                 </ros>
                 <output_type>sensor_msgs/LaserScan</output_type>
-                <frame_name>laser_frame</frame_name>
+                <frame_name>base_laser</frame_name>
             </plugin>
         </sensor>

Commit message: test lidar

File: description/ld19.xacro (robot description, xacro)
@@ -2,5 +2,5 @@
 <robot xmlns:xacro="http://www.ros.org/wiki/xacro"  name="robot">
     <joint name="laser_joint" type="fixed">
-        <parent link="chassis"/>
+        <parent link="base_link"/>
         <child link="base_laser"/>
         <origin xyz="0.07725 0 0.10009" rpy="0 0 ${pi/2}"/>

Commit message: correction

File: description/ld19.xacro (robot description, xacro)
@@ -4,5 +4,5 @@
         <parent link="base_link"/>
         <child link="base_laser"/>
-        <origin xyz="0.07725 0 0.10009" rpy="0 0 ${pi/2}"/>
+        <origin xyz="0.07725 0 0.1051" rpy="0 0 ${pi/2}"/>
     </joint>
     <link name="base_laser">
