Commit message: change in chassis

File: description/robot_core.xacro (robot description, xacro)
@@ -32,5 +32,5 @@
         <origin xyz="0.078185 0 0.0458"/>
             <geometry>
-                <box size="0.15637 0.062 0.0916"/>
+                <box size="0.15637 0.062 0.060"/>
             </geometry>
             <material name="grey"></material>
@@ -39,8 +39,8 @@
         <origin xyz="0.078185 0 0.0458"/>
             <geometry>
-                <box size="0.15637 0.062 0.0916"/>
+                <box size="0.15637 0.062 0.060"/>
             </geometry>
         </collision>
-        <xacro:inertial_box mass="0.567" x="0.15637" y="0.062" z="0.0916">
+        <xacro:inertial_box mass="0.567" x="0.15637" y="0.062" z="0.060">
             <origin xyz="0.078185 0 0.0458" rpy="0 0 0"/>
         </xacro:inertial_box>

Commit message: slam started

File: description/robot_core.xacro (robot description, xacro)
@@ -20,5 +20,14 @@
         <color rgba="0.8588235294117647 0.7058823529411765 0.047058823529411764 1.0"/>
     </material>
+      <!-- BASE LINK-->
     <link name="base_link">
+    </link>
+     <!-- BASE_FOOTPRINT LINK -->
+    <joint name="base_footprint_joint" type="fixed">
+        <parent link="base_link"/>
+        <child link="base_footprint"/>
+        <origin xyz="0 0 0" rpy="0 0 0"/>
+    </joint>
+    <link name="base_footprint">
     </link>
     <!-- CHASSIS LINK-->

Commit message: chage base_footprint

File: description/robot_core.xacro (robot description, xacro)
@@ -27,5 +27,5 @@
         <parent link="base_link"/>
         <child link="base_footprint"/>
-        <origin xyz="0 0 0" rpy="0 0 0"/>
+        <origin xyz="0 0 -0.05504" rpy="0 0 0"/>
     </joint>
     <link name="base_footprint">
