Commit message: robot in gazebo done

File: description/robot.urdf.xacro (robot description, xacro)
@@ -2,4 +2,5 @@
 <robot xmlns:xacro="http://www.ros.org/wiki/xacro"  name="robot">
     <xacro:include filename="robot_core.xacro"/>
-    <xacro:include filename="robot_gazebo.gazebo.xacro"/>
+    <xacro:include filename="robot_gazebo_color.gazebo.xacro"/>
+    <xacro:include filename="gazebo_control.xacro"/>
 </robot>

File: description/robot_core.xacro (robot description, xacro)
@@ -56,5 +56,5 @@
         <visual>
             <geometry>
-                <cylinder radius="0.0215" length="0.01775"/>
+                <cylinder radius="0.0225" length="0.01775"/>
             </geometry>
             <material name="black"></material>
@@ -62,5 +62,5 @@
         <collision>
             <geometry>
-                <cylinder radius="0.0215" length="0.01775"/>
+                <cylinder radius="0.0225" length="0.01775"/>
             </geometry>
         </collision>
@@ -79,5 +79,5 @@
         <visual>
             <geometry>
-                <cylinder radius="0.0215" length="0.01775"/>
+                <cylinder radius="0.0225" length="0.01775"/>
             </geometry>
             <material name="black"></material>
@@ -85,5 +85,5 @@
         <collision>
             <geometry>
-                <cylinder radius="0.0215" length="0.01775"/>
+                <cylinder radius="0.0225" length="0.01775"/>
             </geometry>
         </collision>

File: description/robot_gazebo_color.gazebo.xacro (robot description, xacro)
@@ -2,14 +2,16 @@
 <robot xmlns:xacro="http://www.ros.org/wiki/xacro"  name="robot">
     <gazebo reference="chassis">
-        <material>Gazebo/grey</material>
+        <material>Gazebo/Grey</material>
     </gazebo>
     <gazebo reference="left_wheel">
-        <material>Gazebo/black</material>
+        <material>Gazebo/Black</material>
     </gazebo>
     <gazebo reference="right_wheel">
-        <material>Gazebo/black</material>
+        <material>Gazebo/Black</material>
     </gazebo>
     <gazebo reference="caster_wheel">
-        <material>Gazebo/white</material>
+        <material>Gazebo/White</material>
+        <mu1 value="0.00001"></mu1>
+        <mu2 value="0.00001"></mu2>
     </gazebo>
 </robot>

Commit message: with netplan

File: description/robot.urdf.xacro (robot description, xacro)
@@ -4,3 +4,4 @@
     <xacro:include filename="robot_gazebo_color.gazebo.xacro"/>
     <xacro:include filename="gazebo_control.xacro"/>
+    <xacro:include filename="lidar.xacro"/>
 </robot>

File: description/robot_gazebo_color.gazebo.xacro (robot description, xacro)
@@ -15,3 +15,6 @@
         <mu2 value="0.00001"></mu2>
     </gazebo>
+    <gazebo reference="laser_frame">
+        <material>Gazebo/Gold</material>
+    </gazebo>
 </robot>

Commit message: camera added

File: description/robot.urdf.xacro (robot description, xacro)
@@ -5,3 +5,4 @@
     <xacro:include filename="gazebo_control.xacro"/>
     <xacro:include filename="lidar.xacro"/>
+    <xacro:include filename="camera.xacro"/>
 </robot>

File: description/robot_gazebo_color.gazebo.xacro (robot description, xacro)
@@ -18,3 +18,6 @@
         <material>Gazebo/Gold</material>
     </gazebo>
+    <gazebo reference="camera_link">
+        <material>Gazebo/Black</material>
+    </gazebo>
 </robot>

Commit message: ros2_control
need testing

File: description/robot.urdf.xacro (robot description, xacro)
@@ -3,6 +3,7 @@
     <xacro:include filename="robot_core.xacro"/>
     <xacro:include filename="robot_gazebo_color.gazebo.xacro"/>
-    <xacro:include filename="gazebo_control.xacro"/>
+    <!-- <xacro:include filename="gazebo_control.xacro"/> -->
     <xacro:include filename="lidar.xacro"/>
     <xacro:include filename="camera.xacro"/>
+    <xacro:include filename="ros2_control.xacro"/>
 </robot>

File: description/robot_core.xacro (robot description, xacro)
@@ -50,5 +50,5 @@
         <parent link="base_link"/>
         <child link="left_wheel"/>
-        <origin xyz="0 0.05113 0" rpy="-${pi/2} 0 0"/>
+        <origin xyz="0 0.051115 0" rpy="-${pi/2} 0 0"/>
         <axis xyz="0.0 0.0 1"/>
     </joint>
@@ -73,5 +73,5 @@
         <parent link="base_link"/>
         <child link="right_wheel"/>
-        <origin xyz="0 -0.05113 0" rpy="${pi/2} 0 0"/>
+        <origin xyz="0 -0.051115 0" rpy="${pi/2} 0 0"/>
         <axis xyz="0.0 0.0 -1"/>
     </joint>

Commit message: test tf

File: description/robot.urdf.xacro (robot description, xacro)
@@ -11,7 +11,7 @@
         <xacro:include filename="ros2_control.xacro" />
     </xacro:if>
-    <xacro:unless value="$(arg use_ros2_control)">
+    <!-- <xacro:unless value="$(arg use_ros2_control)">
         <xacro:include filename="gazebo_control.xacro" />
-    </xacro:unless>
+    </xacro:unless> -->
     <xacro:include filename="ld19.xacro"/>
 </robot>

File: description/robot_core.xacro (robot description, xacro)
@@ -27,5 +27,5 @@
         <parent link="base_link"/>
         <child link="base_footprint"/>
-        <origin xyz="0 0 -0.05504" rpy="0 0 0"/>
+        <origin xyz="0 0 -0.02961" rpy="0 0 0"/>
     </joint>
     <link name="base_footprint">
